Commit message: fix: align integration scope and shared configuration

File: ros2_ws/src/description/urdf/robot.urdf.xacro (robot description, xacro)
@@ -35,5 +35,5 @@
        위치 · 질량은 가정 -->
   <xacro:arg name="with_accessories" default="true"/>
-  <xacro:arg name="hardware_map" default="$(find description)/config/hardware_map.yaml"/>
+  <xacro:arg name="hardware_map" default="$(find bringup)/config/hardware_map.yaml"/>
   <xacro:arg name="opencr_port" default="auto"/>   <!-- hardware:=opencr 때 포트 바꾸기 — 보드 1장일 때만 (auto = hardware_map.yaml 의 port) -->
   <xacro:arg name="opencr_ports" default="auto"/>  <!-- 보드마다: bus_drive=/tmp/opencr_drive,bus_arm=/tmp/opencr_arm (auto = hardware_map.yaml) -->
@@ -44,5 +44,5 @@
   <!-- base_link 원점 = 조향축 4개의 한가운데, 바퀴축 높이. 단위 m -->
   <xacro:property name="wheel_r" value="0.033"/>       <!-- 바퀴 반지름 (CAD 타이어 33.0 mm, 터틀봇3 바퀴와 같음) -->
-  <xacro:property name="module_x" value="0.112"/>      <!-- 조향축 위치 ±x (bringup/config/controllers.yaml 의 swerve_controller 와 같아야 함!) -->
+  <xacro:property name="module_x" value="0.112"/>      <!-- 조향축 위치 ±x (config/controllers.yaml 의 swerve_controller 와 같아야 함!) -->
   <xacro:property name="module_y" value="0.064"/>      <!-- 조향축 위치 ±y -->
   <xacro:property name="wheel_off" value="0.0269"/>    <!-- 바퀴 중심이 조향축에서 바깥쪽으로 떨어진 거리 (바퀴축 방향) -->

File: ros2_ws/src/description/urdf/ros2_control.xacro (robot description, xacro)
@@ -9,5 +9,5 @@
     gazebo  : Gazebo(gz_ros2_control) 용 자리만 (시뮬레이션 월드 · 실행 설정은 아직 없음)
     opencr  : 플러그인 hardware/OpenCRHardware + OpenCR 펌웨어 firmware/nt_opencr
-              모터 14개 + OpenCR 내장 IMU 를 USB 한 줄로. 패킷 규칙 = docs/hardware.md 4절
+              모터 14개 + OpenCR 내장 IMU 를 USB 한 줄로. 패킷 정의 = firmware/nt_opencr/nt_packet.h
   ★ 이 한 줄만 바뀌고, 컨트롤러 · 스워브 노드 · MoveIt · Nav2 는 전부 그대로다.
   맨 아래 관성 · 충돌 상자 매크로 ⚠ 질량 · 관성은 추정. 실측 물성이 아님
@@ -62,5 +62,5 @@
           <!-- ros2_ws/src/hardware (설명은 opencr_hardware.hpp) -->
           <plugin>hardware/OpenCRHardware</plugin>
-          <!-- 포트: opencr_ports:=bus_drive=/tmp/a,bus_arm=/tmp/b 로 보드마다 바꿈 (가짜 보드 tools/fw_sim 시험 등)
+          <!-- 포트: opencr_ports:=bus_drive=/tmp/a,bus_arm=/tmp/b 로 보드마다 바꿈 (사용자가 명시한 보드별 포트)
                opencr_port:=… (예전 인자) 는 보드가 1장일 때만. 둘 다 auto 면 hardware_map.yaml 의 port -->
           <param name="port_name">${opencr_ports.get(bus['name'], bus['port'] if ('$(arg opencr_port)' == 'auto' or len(hw['buses']) != 1) else '$(arg opencr_port)')}</param>
